File: noise_pcb_power_supply.kicad_sch (KiCad schematic)
At the start: 10 parts, among them J1 Conn_02x05_Odd_Even, U2 LM7805_TO220

Commit message: Title block updates and pdf
Other:
- company: (none) -> Robot Dialogs
- title: (none) -> Noise PCB
Changed lines of the file:
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@@
 (kicad_sch (version 20211123) (generator eeschema)
   (paper "A4")
+  (title_block
+    (title "Noise PCB")
+    (date "2022-01-31")
+    (rev "1.0")
+    (company "Robot Dialogs")
+  )
   (junction (at 183.515 65.405) (diameter 0) (color 0 0 0 0)
   )
